File: 6502_computer.kicad_sch (KiCad schematic)
At the start: 0 parts

Commit message: First board
Parts:
- added C1: 10u, Capacitor_THT:CP_Radial_D4.0mm_P1.50mm, symbol Device:C_Polarized_Small
- added C2, C3: 100n, Capacitor_THT:C_Disc_D5.0mm_W2.5mm_P5.00mm, symbol Device:C_Small
- added D1: POWER, LED_THT:LED_D3.0mm, symbol Device:LED_Small
- added DS1: WC1602A, Display:WC1602A, symbol Display_Character:WC1602A
- added J1: Barrel_Jack_Switch, Connector_BarrelJack:BarrelJack_Horizontal, symbol Connector:Barrel_Jack_Switch
- added J2: Conn_01x16, Connector_PinSocket_2.54mm:PinSocket_1x16_P2.54mm_Vertical, symbol Connector_Generic:Conn_01x16
- added R1: 1k, Resistor_THT:R_Axial_DIN0207_L6.3mm_D2.5mm_P7.62mm_Horizontal, symbol Device:R_Small
- added RV1: 4.7k, Potentiometer_THT:Potentiometer_Vishay_T7-YA_Single_Vertical, symbol Device:R_Potentiometer
- added U1: 6502_mainboard_v2, AK's_Footprints:Mainboard v2, symbol AK's_Library:6502_mainboard_v2
- added U2: W65C22SxP, Package_DIP:DIP-40_W15.24mm, symbol 65xx:W65C22SxP
- added U3: Keyboard_v1, AK's_Footprints:Keyboard v1, symbol AK's_Library:Keyboard_v1
Connections:
- net GND: now also C1.2, C2.2, C3.2, DS1.1 (VSS), DS1.16 (LED(-)), J1.2, J2.2 (Pin_2), R1.2, RV1.1, U1.2 (GND), U2.1 (VSS), U3.2 (GND)
- net VCC: now also C1.1, C2.1, C3.1, D1.2 (A), DS1.15 (LED(+)), DS1.2 (VDD), J1.1, J2.1 (Pin_1), RV1.3, U1.1 (VCC), U2.20 (VCC), U2.24 (CS1), U3.1 (VCC)
- new net: D1.1 (K), R1.1
- new net: DS1.3 (VO), RV1.2
- new net A0: U1.6 (A0), U2.38 (RS0)
- new net A1: U1.7 (A1), U2.37 (RS1)
- new net A2: U1.8 (A2), U2.36 (RS2)
- new net A3: U1.9 (A3), U2.35 (RS3)
- new net CLK: U1.4 (CLK), U2.25 (ϕ2)
- new net CS_VIA: U1.30 (~{IO1}), U2.23 (~{CS2})
- new net D0: U1.22 (D0), U2.33 (D0)
- new net D1: U1.23 (D1), U2.32 (D1)
- new net D2: U1.24 (D2), U2.31 (D2)
- new net D3: U1.25 (D3), U2.30 (D3)
- new net D4: U1.26 (D4), U2.29 (D4)
- new net D5: U1.27 (D5), U2.28 (D5)
- new net D6: U1.28 (D6), U2.27 (D6)
- new net D7: U1.29 (D7), U2.26 (D7)
- new net IRQ_VIA: U1.34 (~{IRQ1}), U2.21 (~{IRQ})
- new net KB_E: U2.5 (PA3), U3.5 (BUS_ENABLE)
- new net KB_IRQ: U2.18 (CB1), U3.3 (IRQ)
- new net KB_VALID: U2.6 (PA4), U3.4 (VALID_PACKET)
- new net LCD_E: DS1.6 (E), U2.2 (PA0)
- new net LCD_RS: DS1.4 (RS), U2.4 (PA2)
- new net LCD_RW: DS1.5 (R/W), U2.3 (PA1)
- new net PB0: DS1.7 (D0), J2.16 (Pin_16), U2.10 (PB0), U3.13 (D0)
- new net PB1: DS1.8 (D1), J2.15 (Pin_15), U2.11 (PB1), U3.12 (D1)
- new net PB2: DS1.9 (D2), J2.14 (Pin_14), U2.12 (PB2), U3.11 (D2)
- new net PB3: DS1.10 (D3), J2.13 (Pin_13), U2.13 (PB3), U3.10 (D3)
- new net PB4: DS1.11 (D4), J2.12 (Pin_12), U2.14 (PB4), U3.9 (D4)
- new net PB5: DS1.12 (D5), J2.11 (Pin_11), U2.15 (PB5), U3.8 (D5)
- new net PB6: DS1.13 (D6), J2.10 (Pin_10), U2.16 (PB6), U3.7 (D6)
- new net PB7: DS1.14 (D7), J2.9 (Pin_9), U2.17 (PB7), U3.6 (D7)
- new net R~{W}: U1.41 (R~{W}), U2.22 (R/~{W})
- new net VIA_CA1: J2.5 (Pin_5), U2.40 (CA1)
- new net VIA_CA2: J2.4 (Pin_4), U2.39 (CA2)
- new net VIA_CB2: J2.3 (Pin_3), U2.19 (CB2)
- new net VIA_PA5: J2.8 (Pin_8), U2.7 (PA5)
- new net VIA_PA6: J2.7 (Pin_7), U2.8 (PA6)
- new net VIA_PA7: J2.6 (Pin_6), U2.9 (PA7)
- new net ~{RST}: U1.3 (~{RST}), U2.34 (~{RES})
- no-connect marks 0 -> 32

Commit message: Update
Parts:
- removed C3: 100n, Capacitor_THT:C_Disc_D5.0mm_W2.5mm_P5.00mm, symbol Device:C_Small
- added J3: Mega, Connector_PinHeader_2.54mm:PinHeader_2x18_P2.54mm_Vertical, symbol Connector_Generic:Conn_02x18_Odd_Even
- added J4: Mega, Connector_PinSocket_2.54mm:PinSocket_1x04_P2.54mm_Vertical, symbol Connector_Generic:Conn_01x04
- added J5: Clock, Connector_PinSocket_2.54mm:PinSocket_1x03_P2.54mm_Vertical, symbol Connector_Generic:Conn_01x03
- added J6: Conn_01x40, Connector_PinSocket_2.54mm:PinSocket_1x40_P2.54mm_Vertical, symbol Connector_Generic:Conn_01x40
- added J7: Conn_01x06, Connector_PinSocket_2.54mm:PinSocket_1x06_P2.54mm_Vertical, symbol Connector_Generic:Conn_01x06
- added J8, J9: Conn_01x02, Connector_PinSocket_2.54mm:PinSocket_1x02_P2.54mm_Vertical, symbol Connector_Generic:Conn_01x02
- RV1: value 4.7k -> 10k
Connections:
- net A0: now also J3.3 (Pin_3), J6.21 (Pin_21)
- net A1: now also J3.4 (Pin_4), J6.20 (Pin_20)
- net A2: now also J3.5 (Pin_5), J6.19 (Pin_19)
- net A3: now also J3.6 (Pin_6), J6.18 (Pin_18)
- net CLK: now also J3.34 (Pin_34), J5.3 (Pin_3), J6.4 (Pin_4)
- net D0: now also J3.30 (Pin_30), J6.29 (Pin_29)
- net D1: now also J3.29 (Pin_29), J6.28 (Pin_28)
- net D2: now also J3.28 (Pin_28), J6.27 (Pin_27)
- net D3: now also J3.27 (Pin_27), J6.26 (Pin_26)
- net D4: now also J3.26 (Pin_26), J6.25 (Pin_25)
- net D5: now also J3.25 (Pin_25), J6.24 (Pin_24)
- net D6: now also J3.24 (Pin_24), J6.23 (Pin_23)
- net D7: now also J3.23 (Pin_23), J6.22 (Pin_22)
- net GND: now also J3.35 (Pin_35), J3.36 (Pin_36), J4.2 (Pin_2), J5.2 (Pin_2), J6.2 (Pin_2), J8.2 (Pin_2), J9.2 (Pin_2)
- net KB_E: now also U2.13 (PB3); no longer U2.5 (PA3)
- net KB_IRQ: now also U2.40 (CA1); no longer U2.18 (CB1)
- net KB_VALID: now also U2.14 (PB4); no longer U2.6 (PA4)
- net LCD_E: now also U2.10 (PB0); no longer U2.2 (PA0)
- net LCD_RS: now also U2.12 (PB2); no longer U2.4 (PA2)
- net LCD_RW: now also U2.11 (PB1); no longer U2.3 (PA1)
- net R~{W}: now also J3.32 (Pin_32), J6.39 (Pin_39)
- net VCC: now also J5.1 (Pin_1), J6.1 (Pin_1), J8.1 (Pin_1), J9.1 (Pin_1)
- net VIA_CA2: now also J2.5 (Pin_5); no longer J2.4 (Pin_4)
- net ~{RST}: now also J3.31 (Pin_31), J6.3 (Pin_3)
- net A4: now reaches U1.10 (A4)
- net A4: now also J3.7 (Pin_7), J6.17 (Pin_17)
- net A5: now reaches U1.11 (A5)
- net A5: now also J3.8 (Pin_8), J6.16 (Pin_16)
- net A6: now reaches U1.12 (A6)
- net A6: now also J3.9 (Pin_9), J6.15 (Pin_15)
- net A7: now reaches U1.13 (A7)
- net A7: now also J3.10 (Pin_10), J6.14 (Pin_14)
- net A8: now reaches U1.14 (A8)
- net A8: now also J3.18 (Pin_18), J6.13 (Pin_13)
- net A9: now reaches U1.15 (A9)
- net A9: now also J3.17 (Pin_17), J6.12 (Pin_12)
- net A10: now reaches U1.16 (A10)
- net A10: now also J3.16 (Pin_16), J6.11 (Pin_11)
- net A11: now reaches U1.17 (A11)
- net A11: now also J3.15 (Pin_15), J6.10 (Pin_10)
- net A12: now reaches U1.18 (A12)
- net A12: now also J3.14 (Pin_14), J6.9 (Pin_9)
- net A13: now reaches U1.19 (A13)
- net A13: now also J3.13 (Pin_13), J6.8 (Pin_8)
- net A14: now reaches U1.20 (A14)
- net A14: now also J3.12 (Pin_12), J6.7 (Pin_7)
- net A15: now reaches U1.21 (A15)
- net A15: now also J3.11 (Pin_11), J6.6 (Pin_6)
- net ~{IO2}: now reaches U1.31 (~{IO2})
- net ~{IO2}: now also J6.32 (Pin_32)
- net ~{IO3}: now reaches U1.32 (~{IO3})
- net ~{IO3}: now also J6.31 (Pin_31)
- net ~{IO4}: now reaches U1.33 (~{IO4})
- net ~{IO4}: now also J6.30 (Pin_30)
- net ~{IRQ2}: now reaches U1.35 (~{IRQ2})
- net ~{IRQ2}: now also J6.35 (Pin_35)
- net ~{IRQ3}: now reaches U1.36 (~{IRQ3})
- net ~{IRQ3}: now also J6.34 (Pin_34)
- net ~{IRQ4}: now reaches U1.37 (~{IRQ4})
- net ~{IRQ4}: now also J6.33 (Pin_33)
- net ~{NMI}: now reaches U1.38 (~{NMI})
- net ~{NMI}: now also J6.36 (Pin_36)
- net ~{WR}: now reaches U1.39 (~{WRITE})
- net ~{WR}: now also J6.37 (Pin_37)
- net ~{RD}: now reaches U1.40 (~{READ})
- net ~{RD}: now also J6.38 (Pin_38)
- net RDY: now reaches U1.42 (RDY)
- net RDY: now also J6.40 (Pin_40)
- net BE: now reaches U1.43 (BE)
- net BE: now also J3.21 (Pin_21), J7.1 (Pin_1)
- net ~{ROMW}: now reaches U1.46 (~{ROMW})
- net ~{ROMW}: now also J3.22 (Pin_22), J7.2 (Pin_2)
- net SYNC: now reaches U1.47 (SYNC)
- net SYNC: now also J3.33 (Pin_33), J7.3 (Pin_3)
- net ~{VP}: now reaches U1.48 (~{VP})
- net ~{VP}: now also J7.4 (Pin_4)
- net ~{ML}: now reaches U1.49 (~{ML})
- net ~{ML}: now also J7.5 (Pin_5)
- net ~{CLK}: now reaches U1.5 (~{CLK})
- net ~{CLK}: now also J6.5 (Pin_5)
- net ~{SO}: now reaches U1.50 (~{SO})
- net ~{SO}: now also J7.6 (Pin_6)
- net CS_VIA renamed ~{CS_VIA}
- net IRQ_VIA renamed ~{IRQ_VIA}
- net PB0 renamed PA0
- net PA0: now also U2.2 (PA0); no longer U2.10 (PB0)
- net PB1 renamed PA1
- net PA1: now also U2.3 (PA1); no longer U2.11 (PB1)
- net PB2 renamed PA2
- net PA2: now also U2.4 (PA2); no longer U2.12 (PB2)
- net PB3 renamed PA3
- net PA3: now also U2.5 (PA3); no longer U2.13 (PB3)
- net PB4 renamed PA4
- net PA4: now also U2.6 (PA4); no longer U2.14 (PB4)
- net PB5 renamed PA5
- net PA5: now also U2.7 (PA5); no longer U2.15 (PB5)
- net PB6 renamed PA6
- net PA6: now also U2.8 (PA6); no longer U2.16 (PB6)
- net PB7 renamed PA7
- net PA7: now also U2.9 (PA7); no longer U2.17 (PB7)
- removed net VIA_CA1: J2.5 (Pin_5), U2.40 (CA1)
- net VIA_PA5 renamed VIA_PB5
- net VIA_PB5: now also U2.15 (PB5); no longer U2.7 (PA5)
- net VIA_PA6 renamed VIA_PB6
- net VIA_PB6: now also U2.16 (PB6); no longer U2.8 (PA6)
- net VIA_PA7 renamed VIA_PB7
- net VIA_PB7: now also U2.17 (PB7); no longer U2.9 (PA7)
- new net +5V(MEGA): J3.1 (Pin_1), J3.2 (Pin_2), J4.1 (Pin_1)
- new net MEGA_PD7: J3.19 (Pin_19), J4.4 (Pin_4)
- new net MEGA_PG2: J3.20 (Pin_20), J4.3 (Pin_3)
- new net VIA_CB1: J2.4 (Pin_4), U2.18 (CB1)
- no-connect marks 32 -> 3
Other:
- moved on the sheet: DS1, J2, RV1, U2, U3

Commit message: Update
Parts:
- U1: symbol AK's_Library:6502_mainboard_v2 -> 6502_computer:6502_mainboard_v2
- U2: symbol 65xx:W65C22SxP -> 6502_computer:W65C22SxP
- U3: symbol AK's_Library:Keyboard_v1 -> 6502_computer:Keyboard_v1
Connections:
- net A0: now also J3.4 (Pin_4); no longer J3.3 (Pin_3)
- net A1: now also J3.3 (Pin_3); no longer J3.4 (Pin_4)
- net A10: now also J3.15 (Pin_15); no longer J3.16 (Pin_16)
- net A11: now also J3.16 (Pin_16); no longer J3.15 (Pin_15)
- net A12: now also J3.13 (Pin_13); no longer J3.14 (Pin_14)
- net A13: now also J3.14 (Pin_14); no longer J3.13 (Pin_13)
- net A14: now also J3.11 (Pin_11); no longer J3.12 (Pin_12)
- net A15: now also J3.12 (Pin_12); no longer J3.11 (Pin_11)
- net A2: now also J3.6 (Pin_6); no longer J3.5 (Pin_5)
- net A3: now also J3.5 (Pin_5); no longer J3.6 (Pin_6)
- net A4: now also J3.8 (Pin_8); no longer J3.7 (Pin_7)
- net A5: now also J3.7 (Pin_7); no longer J3.8 (Pin_8)
- net A6: now also J3.10 (Pin_10); no longer J3.9 (Pin_9)
- net A7: now also J3.9 (Pin_9); no longer J3.10 (Pin_10)
- net A8: now also J3.17 (Pin_17); no longer J3.18 (Pin_18)
- net A9: now also J3.18 (Pin_18); no longer J3.17 (Pin_17)
- net BE: now also J3.22 (Pin_22); no longer J3.21 (Pin_21)
- net CLK: now also J3.33 (Pin_33); no longer J3.34 (Pin_34)
- net D0: now also J3.29 (Pin_29); no longer J3.30 (Pin_30)
- net D1: now also J3.30 (Pin_30); no longer J3.29 (Pin_29)
- net D2: now also J3.27 (Pin_27); no longer J3.28 (Pin_28)
- net D3: now also J3.28 (Pin_28); no longer J3.27 (Pin_27)
- net D4: now also J3.25 (Pin_25); no longer J3.26 (Pin_26)
- net D5: now also J3.26 (Pin_26); no longer J3.25 (Pin_25)
- net D6: now also J3.23 (Pin_23); no longer J3.24 (Pin_24)
- net D7: now also J3.24 (Pin_24); no longer J3.23 (Pin_23)
- net MEGA_PD7: now also J3.20 (Pin_20); no longer J3.19 (Pin_19)
- net MEGA_PG2: now also J3.19 (Pin_19); no longer J3.20 (Pin_20)
- net R~{W}: now also J3.31 (Pin_31); no longer J3.32 (Pin_32)
- net SYNC: now also J3.34 (Pin_34); no longer J3.33 (Pin_33)
- net ~{ROMW}: now also J3.21 (Pin_21); no longer J3.22 (Pin_22)
- net ~{RST}: now also J3.32 (Pin_32); no longer J3.31 (Pin_31)

Commit message: Update
Other:
- title: Project Title -> 6502 computer
Changed lines of the file:
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@@
   (paper "A4")
   (title_block
-    (title "Project Title")
-    (date "Date")
-    (rev "REV")
-    (comment 2 "<REPO-URL>")
+    (title "6502 computer")
+    (date "2023-02-20")
+    (rev "1")
+    (comment 2 "https://github.com/adrienkohlbecker/6502_computer")
     (comment 3 "Licensed under CERN-OHL-W v2")
     (comment 4 "Copyright © 2022 Adrien Kohlbecker")
